Commit message: Fixed up metapackage and moved general ridgeback manipulation components to a dedicated package

File: ridgeback_iiwa_description/urdf/ridgeback_iiwa_14_description.urdf.xacro (robot description, xacro)
@@ -3,5 +3,5 @@
   <xacro:include filename="$(find iiwa_description)/urdf/materials.xacro" />
   <xacro:include filename="$(find iiwa_description)/urdf/iiwa14.xacro"/>
-  <xacro:include filename="$(find ridgeback_manipulation)/urdf/hams.urdf.xacro"/>
+  <xacro:include filename="$(find ridgeback_manipulation_description)/urdf/hams.urdf.xacro"/>
   <xacro:arg name="hardware_interface" default="PositionJointInterface"/>
   <xacro:arg name="robot_name" default="iiwa"/>

File: ridgeback_iiwa_description/urdf/ridgeback_iiwa_7_description.urdf.xacro (robot description, xacro)
@@ -3,5 +3,5 @@
   <xacro:include filename="$(find iiwa_description)/urdf/materials.xacro" />
   <xacro:include filename="$(find iiwa_description)/urdf/iiwa7.xacro"/>
-  <xacro:include filename="$(find ridgeback_manipulation)/urdf/hams.urdf.xacro"/>
+  <xacro:include filename="$(find ridgeback_manipulation_description)/urdf/hams.urdf.xacro"/>
   <xacro:arg name="hardware_interface" default="PositionJointInterface"/>
   <xacro:arg name="robot_name" default="iiwa"/>

File: ridgeback_manipulation_description/urdf/hams.urdf.xacro (robot description, xacro)
@@ -5,5 +5,5 @@
     <visual>
       <geometry>
-        <mesh filename="package://ridgeback_manipulation/meshes/hams-table-top.stl" />
+        <mesh filename="package://ridgeback_manipulation_description/meshes/hams-table-top.stl" />
       </geometry>
       <material name="black" />
@@ -12,5 +12,5 @@
       <origin xyz="0 0 0" rpy="0 0 0"/>
       <geometry>
-        <mesh filename="package://ridgeback_manipulation/meshes/hams-table-top.stl" />
+        <mesh filename="package://ridgeback_manipulation_description/meshes/hams-table-top.stl" />
       </geometry>
     </collision>
@@ -19,5 +19,5 @@
     <visual>
       <geometry>
-        <mesh filename="package://ridgeback_manipulation/meshes/hams-table-legs.stl" />
+        <mesh filename="package://ridgeback_manipulation_description/meshes/hams-table-legs.stl" />
       </geometry>
       <material name="light_grey" />
@@ -26,5 +26,5 @@
       <origin xyz="0 0 0" rpy="0 0 0"/>
       <geometry>
-        <mesh filename="package://ridgeback_manipulation/meshes/hams-table-legs.stl" />
+        <mesh filename="package://ridgeback_manipulation_description/meshes/hams-table-legs.stl" />
       </geometry>
     </collision>
@@ -43,5 +43,5 @@
     <visual>
       <geometry>
-        <mesh filename="package://ridgeback_manipulation/meshes/hams-arm-mount.stl" />
+        <mesh filename="package://ridgeback_manipulation_description/meshes/hams-arm-mount.stl" />
       </geometry>
       <material name="black" />
@@ -50,5 +50,5 @@
       <origin xyz="0 0 0" rpy="0 0 0"/>
       <geometry>
-        <mesh filename="package://ridgeback_manipulation/meshes/hams-arm-mount.stl" />
+        <mesh filename="package://ridgeback_manipulation_description/meshes/hams-arm-mount.stl" />
       </geometry>
     </collision>
