Commit message: Updated descriptions for 2.2.  Remade and renamed moveit configs

File: ridgeback_kinova_description/urdf/ridgeback_gen3_description.urdf.xacro (robot description, xacro)
@@ -1,9 +1,16 @@
 <?xml version="1.0"?>
 <robot xmlns:xacro="http://ros.org/wiki/xacro">
-  <xacro:include filename="$(find kortex_description)/robots/gen3.xacro" />
+  <xacro:arg name="arm" default="gen3" />
+  <xacro:arg name="dof" default="7" />
+  <xacro:arg name="vision" default="true" />
+  <xacro:arg name="gripper" default="" />
+  <xacro:arg name="sim" default="false" />
+  <xacro:arg name="prefix" default="kinova_arm_" />
+  <xacro:include filename="$(find kortex_description)/robots/kortex_robot.xacro" />
+  <xacro:load_robot arm="$(arg arm)" gripper="$(arg gripper)" dof="$(arg dof)" vision="$(arg vision)" sim="$(arg sim)" prefix="$(arg prefix)" />
   <joint name="arm_mount_joint" type="fixed">
     <origin xyz="$(optenv RIDGEBACK_KINOVA_XYZ 0.21 0 0)" rpy="$(optenv RIDGEBACK_KINOVA_RPY 0 0 0)" />
     <parent link="mid_mount" />
-    <child link="arm_base_link" />
+    <child link="kinova_arm_base_link" />
   </joint>
 </robot>

File: ridgeback_kinova_description/urdf/ridgeback_gen3_robotiq_2f_140_description.urdf.xacro (robot description, xacro)
@@ -4,5 +4,5 @@
   <xacro:arg name="dof" default="7" />
   <xacro:arg name="vision" default="true" />
-  <xacro:arg name="gripper" default="robotiq_2f_85" />
+  <xacro:arg name="gripper" default="robotiq_2f_140" />
   <xacro:arg name="sim" default="false" />
   <xacro:arg name="prefix" default="kinova_arm_" />
