Commit message: Add the RIDGEBACK_HAMS_ANGLE envar to allow rotating the HAMS mount on the ridgeback. Change the arm mounting plate to be a child of the tabletop link, rather than a child of base_link so it rotates correctly too

File: ridgeback_manipulation_description/urdf/hams.urdf.xacro (robot description, xacro)
@@ -33,10 +33,10 @@
     <parent link="mid_mount" />
     <child link="table_top_link" />
-    <origin xyz="0 0 0.60635" rpy="0 0 0"/>
+    <origin xyz="0 0 0.60635" rpy="0 0 $(optenv RIDGEBACK_HAMS_ANGLE 0)"/>
   </joint>
   <joint name="table_legs_joint" type="fixed">
     <parent link="mid_mount" />
     <child link="table_legs_link" />
-    <origin xyz="0 0 0.60635" rpy="0 0 0"/>
+    <origin xyz="0 0 0.60635" rpy="0 0 $(optenv RIDGEBACK_HAMS_ANGLE 0)"/>
   </joint>
   <link name="arm_mount_link">
@@ -54,8 +54,9 @@
     </collision>
   </link>
+  <xacro:property name="arm_height" value="$(optenv RIDGEBACK_ARM_HEIGHT 0.31)" />
   <joint name="arm_mount_joint" type="fixed">
-    <parent link="mid_mount" />
+    <parent link="table_top_link" />
     <child link="arm_mount_link" />
-    <origin xyz="-.27913 0 $(optenv RIDGEBACK_ARM_HEIGHT 0.31)" rpy="0 0 $(optenv RIDGEBACK_ARM_ANGLE 0.0)"/>
+    <origin xyz="-.27913 0 -${0.60635 - arm_height}" rpy="0 0 $(optenv RIDGEBACK_ARM_ANGLE 0.0)"/>
   </joint>
 </robot>
