Commit message: Changed path to FAMS meshes, was pointing at custom repository

File: ridgeback_manipulation_description/urdf/fams.urdf.xacro (robot description, xacro)
@@ -6,5 +6,5 @@
       <origin xyz="0 0 0" rpy="0 0 0"/>
       <geometry>
-        <mesh filename="package://gnr91_ridgeback/meshes/bar.stl"/>
+        <mesh filename="package://ridgeback_manipulation_description/meshes/fams-table-leg.stl"/>
       </geometry>
       <material name="light_grey"/>
@@ -21,5 +21,5 @@
       <origin xyz="0 0 0" rpy="0 0 0"/>
       <geometry>
-        <mesh filename="package://gnr91_ridgeback/meshes/bar.stl"/>
+        <mesh filename="package://ridgeback_manipulation_description/meshes/fams-table-leg.stl"/>
       </geometry>
       <material name="light_grey"/>
@@ -36,5 +36,5 @@
       <origin xyz="0 0 0" rpy="0 0 0"/>
       <geometry>
-        <mesh filename="package://gnr91_ridgeback/meshes/bar.stl"/>
+        <mesh filename="package://ridgeback_manipulation_description/meshes/fams-table-leg.stl"/>
       </geometry>
       <material name="light_grey"/>
@@ -51,5 +51,5 @@
       <origin xyz="0 0 0" rpy="0 0 0"/>
       <geometry>
-        <mesh filename="package://gnr91_ridgeback/meshes/bar.stl"/>
+        <mesh filename="package://ridgeback_manipulation_description/meshes/fams-table-leg.stl"/>
       </geometry>
       <material name="light_grey"/>
@@ -66,5 +66,5 @@
       <origin xyz="0 0 0" rpy="0 0 0"/>
       <geometry>
-        <mesh filename="package://gnr91_ridgeback/meshes/bar.stl"/>
+        <mesh filename="package://ridgeback_manipulation_description/meshes/fams-table-leg.stl"/>
       </geometry>
       <material name="light_grey"/>
@@ -81,5 +81,5 @@
       <origin xyz="0 0 0" rpy="0 0 0"/>
       <geometry>
-        <mesh filename="package://gnr91_ridgeback/meshes/bar.stl"/>
+        <mesh filename="package://ridgeback_manipulation_description/meshes/fams-table-leg.stl"/>
       </geometry>
       <material name="light_grey"/>
@@ -96,5 +96,5 @@
       <origin xyz="0 0 0" rpy="0 0 0"/>
       <geometry>
-        <mesh filename="package://gnr91_ridgeback/meshes/bar.stl"/>
+        <mesh filename="package://ridgeback_manipulation_description/meshes/fams-table-leg.stl"/>
       </geometry>
       <material name="light_grey"/>
@@ -111,5 +111,5 @@
       <origin xyz="0 0 0" rpy="0 0 0"/>
       <geometry>
-        <mesh filename="package://gnr91_ridgeback/meshes/bar.stl"/>
+        <mesh filename="package://ridgeback_manipulation_description/meshes/fams-table-leg.stl"/>
       </geometry>
       <material name="light_grey"/>
