Commit message: Aded RIDGEBACK_FRANKA_PARENT environment variable to define the parent link of the Panda arm

File: ridgeback_franka_description/urdf/ridgeback_panda_description.urdf.xacro (robot description, xacro)
@@ -2,5 +2,5 @@
 <robot xmlns:xacro="http://ros.org/wiki/xacro">
   <joint name="arm_mount_joint" type="fixed">
-    <parent link="mid_mount" />
+    <parent link="$(optenv RIDGEBACK_FRANKA_PARENT mid_mount)" />
     <child link="franka_mount_link" />
     <origin xyz="$(optenv RIDGEBACK_FRANKA_XYZ 0.21 0.0 0.0)" rpy="$(optenv RIDGEBACK_FRANKA_RPY 0 0 0)"/>
