Commit message: Change default mount link of UR arms to mid_mount

File: ridgeback_ur_description/urdf/ridgeback_ur10_description.urdf.xacro (robot description, xacro)
@@ -3,7 +3,7 @@
   <xacro:include filename="$(find ur_description)/urdf/inc/ur10_macro.xacro" />
   <joint name="arm_mount_joint" type="fixed">
-    <parent link="top_plate_front_link" />
+    <parent link="mid_mount" />
     <child link="ur_arm_base_link" />
-    <origin xyz="$(optenv RIDGEBACK_UR_XYZ -0.105 0.0 0.0)" rpy="$(optenv RIDGEBACK_UR_RPY 0 0 3.1415927)"/>
+    <origin xyz="$(optenv RIDGEBACK_UR_XYZ 0 0 0)" rpy="$(optenv RIDGEBACK_UR_RPY 0 0 0)"/>
   </joint>
   <xacro:ur10_robot prefix="ur_arm_" />

File: ridgeback_ur_description/urdf/ridgeback_ur10_e_description.urdf.xacro (robot description, xacro)
@@ -3,7 +3,7 @@
   <xacro:include filename="$(find ur_description)/urdf/inc/ur10e_macro.xacro" />
   <joint name="arm_mount_joint" type="fixed">
-    <parent link="top_plate_front_link" />
+    <parent link="mid_mount" />
     <child link="ur_arm_base_link" />
-    <origin xyz="$(optenv RIDGEBACK_UR_XYZ -0.105 0.0 0.0)" rpy="$(optenv RIDGEBACK_UR_RPY 0 0 3.1415927)"/>
+    <origin xyz="$(optenv RIDGEBACK_UR_XYZ 0 0 0)" rpy="$(optenv RIDGEBACK_UR_RPY 0 0 0)"/>
   </joint>
   <xacro:ur10e_robot prefix="ur_arm_" />

File: ridgeback_ur_description/urdf/ridgeback_ur5_description.urdf.xacro (robot description, xacro)
@@ -3,7 +3,7 @@
   <xacro:include filename="$(find ur_description)/urdf/inc/ur5_macro.xacro" />
   <joint name="arm_mount_joint" type="fixed">
-    <parent link="top_plate_front_link" />
+    <parent link="mid_mount" />
     <child link="ur_arm_base_link" />
-    <origin xyz="$(optenv RIDGEBACK_UR_XYZ -0.105 0.0 0.0)" rpy="$(optenv RIDGEBACK_UR_RPY 0 0 3.1415927)"/>
+    <origin xyz="$(optenv RIDGEBACK_UR_XYZ 0 0 0)" rpy="$(optenv RIDGEBACK_UR_RPY 0 0 0)"/>
   </joint>
   <xacro:ur5_robot prefix="ur_arm_" />

File: ridgeback_ur_description/urdf/ridgeback_ur5_e_description.urdf.xacro (robot description, xacro)
@@ -3,7 +3,7 @@
   <xacro:include filename="$(find ur_description)/urdf/inc/ur5e_macro.xacro" />
   <joint name="arm_mount_joint" type="fixed">
-    <parent link="top_plate_front_link" />
+    <parent link="mid_mount" />
     <child link="ur_arm_base_link" />
-    <origin xyz="$(optenv RIDGEBACK_UR_XYZ -0.105 0.0 0.0)" rpy="$(optenv RIDGEBACK_UR_RPY 0 0 3.1415927)"/>
+    <origin xyz="$(optenv RIDGEBACK_UR_XYZ 0 0 0)" rpy="$(optenv RIDGEBACK_UR_RPY 0 0 0)"/>
   </joint>
   <xacro:ur5e_robot prefix="ur_arm_" />
