Commit message: Update UR arm packages (as per husky_manipulation)

File: ridgeback_ur_description/urdf/ridgeback_dual_ur10_description.urdf.xacro (robot description, xacro)
@@ -1,19 +1,16 @@
 <?xml version="1.0"?>
 <robot xmlns:xacro="http://ros.org/wiki/xacro">
+  <xacro:include filename="$(find ur_description)/urdf/inc/ur10_macro.xacro" />
   <joint name="left_arm_mount_joint" type="fixed">
-    <parent link="mid_mount" />
+    <parent link="left_arm_bulkhead_link" />
     <child link="left_ur_arm_base_link" />
-    <origin xyz="$(optenv RIDGEBACK_LEFT_UR_XYZ 0.21 0.20 0.0)" rpy="$(optenv RIDGEBACK_LEFT_UR_RPY 0 0 0)"/>
+    <origin xyz="$(optenv RIDGEBACK_LEFT_UR_XYZ 0 0 0)" rpy="$(optenv RIDGEBACK_LEFT_UR_RPY 0 0 0)"/>
   </joint>
   <joint name="right_arm_mount_joint" type="fixed">
-    <parent link="mid_mount" />
+    <parent link="right_arm_bulkhead_link" />
     <child link="right_ur_arm_base_link" />
-    <origin xyz="$(optenv RIDGEBACK_RIGHT_UR_XYZ 0.21 -0.20 0.0)" rpy="$(optenv RIDGEBACK_RIGHT_UR_RPY 0 0 0)"/>
+    <origin xyz="$(optenv RIDGEBACK_RIGHT_UR_XYZ 0 0 0)" rpy="$(optenv RIDGEBACK_RIGHT_UR_RPY 0 0 0)"/>
   </joint>
-  <xacro:include filename="$(find ur_description)/urdf/ur10.urdf.xacro" />
-  <xacro:arg name="kinematics_config" default="$(find ur_description)/config/ur10_default.yaml" />
-  <xacro:arg name="transmission_hw_interface" default="hardware_interface/PositionJointInterface"/>
-  <xacro:include filename="$(find ur_description)/urdf/common.gazebo.xacro" />
-  <xacro:ur10_robot prefix="left_ur_arm_" joint_limited="true" kinematics_file="${load_yaml('$(arg kinematics_config)')}" />
-  <xacro:ur10_robot prefix="right_ur_arm_" joint_limited="true" kinematics_file="${load_yaml('$(arg kinematics_config)')}" />
+  <xacro:ur10_robot prefix="right_ur_arm_" />
+  <xacro:ur10_robot prefix="left_ur_arm_" />
 </robot>

File: ridgeback_ur_description/urdf/ridgeback_dual_ur10_e_description.urdf.xacro (robot description, xacro)
@@ -1,19 +1,16 @@
 <?xml version="1.0"?>
 <robot xmlns:xacro="http://ros.org/wiki/xacro">
+  <xacro:include filename="$(find ur_description)/urdf/inc/ur10e_macro.xacro" />
   <joint name="left_arm_mount_joint" type="fixed">
-    <parent link="mid_mount" />
+    <parent link="left_arm_bulkhead_link" />
     <child link="left_ur_arm_base_link" />
-    <origin xyz="$(optenv RIDGEBACK_LEFT_UR_XYZ 0.21 0.20 0.0)" rpy="$(optenv RIDGEBACK_LEFT_UR_RPY 0 0 0)"/>
+    <origin xyz="$(optenv RIDGEBACK_LEFT_UR_XYZ 0 0 0)" rpy="$(optenv RIDGEBACK_LEFT_UR_RPY 0 0 0)"/>
   </joint>
   <joint name="right_arm_mount_joint" type="fixed">
-    <parent link="mid_mount" />
+    <parent link="right_arm_bulkhead_link" />
     <child link="right_ur_arm_base_link" />
-    <origin xyz="$(optenv RIDGEBACK_RIGHT_UR_XYZ 0.21 -0.20 0.0)" rpy="$(optenv RIDGEBACK_RIGHT_UR_RPY 0 0 0)"/>
+    <origin xyz="$(optenv RIDGEBACK_RIGHT_UR_XYZ 0 0 0)" rpy="$(optenv RIDGEBACK_RIGHT_UR_RPY 0 0 0)"/>
   </joint>
-  <xacro:include filename="$(find ur_e_description)/urdf/ur10e.urdf.xacro" />
-  <xacro:arg name="kinematics_config" default="$(find ur_description)/config/ur10_e_default.yaml" />
-  <xacro:arg name="transmission_hw_interface" default="hardware_interface/PositionJointInterface"/>
-  <xacro:include filename="$(find ur_e_description)/urdf/common.gazebo.xacro" />
-  <xacro:ur10e_robot prefix="left_ur_arm_" joint_limited="true" kinematics_file="${load_yaml('$(arg kinematics_config)')}" />
-  <xacro:ur10e_robot prefix="right_ur_arm_" joint_limited="true" kinematics_file="${load_yaml('$(arg kinematics_config)')}" />
+  <xacro:ur10e_robot prefix="right_ur_arm_" />
+  <xacro:ur10e_robot prefix="left_ur_arm_" />
 </robot>

File: ridgeback_ur_description/urdf/ridgeback_dual_ur5_description.urdf.xacro (robot description, xacro)
@@ -1,19 +1,16 @@
 <?xml version="1.0"?>
 <robot xmlns:xacro="http://ros.org/wiki/xacro">
+  <xacro:include filename="$(find ur_description)/urdf/inc/ur5_macro.xacro" />
   <joint name="left_arm_mount_joint" type="fixed">
-    <parent link="mid_mount" />
+    <parent link="left_arm_bulkhead_link" />
     <child link="left_ur_arm_base_link" />
-    <origin xyz="$(optenv RIDGEBACK_LEFT_UR_XYZ 0.21 0.20 0.0)" rpy="$(optenv RIDGEBACK_LEFT_UR_RPY 0 0 0)"/>
+    <origin xyz="$(optenv RIDGEBACK_LEFT_UR_XYZ 0 0 0)" rpy="$(optenv RIDGEBACK_LEFT_UR_RPY 0 0 0)"/>
   </joint>
   <joint name="right_arm_mount_joint" type="fixed">
-    <parent link="mid_mount" />
+    <parent link="right_arm_bulkhead_link" />
     <child link="right_ur_arm_base_link" />
-    <origin xyz="$(optenv RIDGEBACK_RIGHT_UR_XYZ 0.21 -0.20 0.0)" rpy="$(optenv RIDGEBACK_RIGHT_UR_RPY 0 0 0)"/>
+    <origin xyz="$(optenv RIDGEBACK_RIGHT_UR_XYZ 0 0 0)" rpy="$(optenv RIDGEBACK_RIGHT_UR_RPY 0 0 0)"/>
   </joint>
-  <xacro:include filename="$(find ur_description)/urdf/ur5.urdf.xacro" />
-  <xacro:arg name="kinematics_config" default="$(find ur_description)/config/ur5_default.yaml" />
-  <xacro:arg name="transmission_hw_interface" default="hardware_interface/PositionJointInterface"/>
-  <xacro:include filename="$(find ur_description)/urdf/common.gazebo.xacro" />
-  <xacro:ur5_robot prefix="left_ur_arm_" joint_limited="true" kinematics_file="${load_yaml('$(arg kinematics_config)')}" />
-  <xacro:ur5_robot prefix="right_ur_arm_" joint_limited="true" kinematics_file="${load_yaml('$(arg kinematics_config)')}" />
+  <xacro:ur5_robot prefix="right_ur_arm_" />
+  <xacro:ur5_robot prefix="left_ur_arm_" />
 </robot>

File: ridgeback_ur_description/urdf/ridgeback_dual_ur5_e_description.urdf.xacro (robot description, xacro)
@@ -1,19 +1,16 @@
 <?xml version="1.0"?>
 <robot xmlns:xacro="http://ros.org/wiki/xacro">
+  <xacro:include filename="$(find ur_description)/urdf/inc/ur5e_macro.xacro" />
   <joint name="left_arm_mount_joint" type="fixed">
-    <parent link="mid_mount" />
+    <parent link="left_arm_bulkhead_link" />
     <child link="left_ur_arm_base_link" />
-    <origin xyz="$(optenv RIDGEBACK_LEFT_UR_XYZ 0.21 0.20 0.0)" rpy="$(optenv RIDGEBACK_LEFT_UR_RPY 0 0 0)"/>
+    <origin xyz="$(optenv RIDGEBACK_LEFT_UR_XYZ 0 0 0)" rpy="$(optenv RIDGEBACK_LEFT_UR_RPY 0 0 0)"/>
   </joint>
   <joint name="right_arm_mount_joint" type="fixed">
-    <parent link="mid_mount" />
+    <parent link="right_arm_bulkhead_link" />
     <child link="right_ur_arm_base_link" />
-    <origin xyz="$(optenv RIDGEBACK_RIGHT_UR_XYZ 0.21 -0.20 0.0)" rpy="$(optenv RIDGEBACK_RIGHT_UR_RPY 0 0 0)"/>
+    <origin xyz="$(optenv RIDGEBACK_RIGHT_UR_XYZ 0 0 0)" rpy="$(optenv RIDGEBACK_RIGHT_UR_RPY 0 0 0)"/>
   </joint>
-  <xacro:include filename="$(find ur_e_description)/urdf/ur5e.urdf.xacro" />
-  <xacro:arg name="kinematics_config" default="$(find ur_description)/config/ur5_e_default.yaml" />
-  <xacro:arg name="transmission_hw_interface" default="hardware_interface/PositionJointInterface"/>
-  <xacro:include filename="$(find ur_e_description)/urdf/common.gazebo.xacro" />
-  <xacro:ur5e_robot prefix="left_ur_arm_" joint_limited="true" kinematics_file="${load_yaml('$(arg kinematics_config)')}" />
-  <xacro:ur5e_robot prefix="right_ur_arm_" joint_limited="true" kinematics_file="${load_yaml('$(arg kinematics_config)')}" />
+  <xacro:ur5e_robot prefix="right_ur_arm_" />
+  <xacro:ur5e_robot prefix="left_ur_arm_" />
 </robot>

File: ridgeback_ur_description/urdf/ridgeback_ur10_description.urdf.xacro (robot description, xacro)
@@ -1,13 +1,10 @@
 <?xml version="1.0"?>
 <robot xmlns:xacro="http://ros.org/wiki/xacro">
+  <xacro:include filename="$(find ur_description)/urdf/inc/ur10_macro.xacro" />
   <joint name="arm_mount_joint" type="fixed">
-    <parent link="mid_mount" />
+    <parent link="top_plate_front_link" />
     <child link="ur_arm_base_link" />
-    <origin xyz="$(optenv RIDGEBACK_UR_XYZ 0.21 0.0 0.0)" rpy="$(optenv RIDGEBACK_UR_RPY 0 0 0)"/>
+    <origin xyz="$(optenv RIDGEBACK_UR_XYZ -0.105 0.0 0.0)" rpy="$(optenv RIDGEBACK_UR_RPY 0 0 3.1415927)"/>
   </joint>
-  <xacro:include filename="$(find ur_description)/urdf/ur10.urdf.xacro" />
-  <xacro:arg name="kinematics_config" default="$(find ur_description)/config/ur10_default.yaml" />
-  <xacro:arg name="transmission_hw_interface" default="hardware_interface/PositionJointInterface"/>
-  <xacro:include filename="$(find ur_description)/urdf/common.gazebo.xacro" />
-  <xacro:ur10_robot prefix="ur_arm_" joint_limited="true" kinematics_file="${load_yaml('$(arg kinematics_config)')}" />
+  <xacro:ur10_robot prefix="ur_arm_" />
 </robot>

File: ridgeback_ur_description/urdf/ridgeback_ur10_e_description.urdf.xacro (robot description, xacro)
@@ -1,13 +1,10 @@
 <?xml version="1.0"?>
 <robot xmlns:xacro="http://ros.org/wiki/xacro">
+  <xacro:include filename="$(find ur_description)/urdf/inc/ur10e_macro.xacro" />
   <joint name="arm_mount_joint" type="fixed">
-    <parent link="mid_mount" />
+    <parent link="top_plate_front_link" />
     <child link="ur_arm_base_link" />
-    <origin xyz="$(optenv RIDGEBACK_UR_XYZ 0.21 0.0 0.0)" rpy="$(optenv RIDGEBACK_UR_RPY 0 0 0)"/>
+    <origin xyz="$(optenv RIDGEBACK_UR_XYZ -0.105 0.0 0.0)" rpy="$(optenv RIDGEBACK_UR_RPY 0 0 3.1415927)"/>
   </joint>
-  <xacro:include filename="$(find ur_e_description)/urdf/ur10e.urdf.xacro" />
-  <xacro:arg name="kinematics_config" default="$(find ur_description)/config/ur10_e_default.yaml" />
-  <xacro:arg name="transmission_hw_interface" default="hardware_interface/PositionJointInterface"/>
-  <xacro:include filename="$(find ur_e_description)/urdf/common.gazebo.xacro" />
-  <xacro:ur10e_robot prefix="ur_arm_" joint_limited="true" kinematics_file="${load_yaml('$(arg kinematics_config)')}" />
+  <xacro:ur10e_robot prefix="ur_arm_" />
 </robot>

File: ridgeback_ur_description/urdf/ridgeback_ur5_description.urdf.xacro (robot description, xacro)
@@ -1,13 +1,10 @@
 <?xml version="1.0"?>
 <robot xmlns:xacro="http://ros.org/wiki/xacro">
+  <xacro:include filename="$(find ur_description)/urdf/inc/ur5_macro.xacro" />
   <joint name="arm_mount_joint" type="fixed">
-    <parent link="mid_mount" />
+    <parent link="top_plate_front_link" />
     <child link="ur_arm_base_link" />
-    <origin xyz="$(optenv RIDGEBACK_UR_XYZ 0.21 0.0 0.0)" rpy="$(optenv RIDGEBACK_UR_RPY 0 0 0)"/>
+    <origin xyz="$(optenv RIDGEBACK_UR_XYZ -0.105 0.0 0.0)" rpy="$(optenv RIDGEBACK_UR_RPY 0 0 3.1415927)"/>
   </joint>
-  <xacro:include filename="$(find ur_description)/urdf/ur5.urdf.xacro" />
-  <xacro:arg name="kinematics_config" default="$(find ur_description)/config/ur5_default.yaml" />
-  <xacro:arg name="transmission_hw_interface" default="hardware_interface/PositionJointInterface"/>
-  <xacro:include filename="$(find ur_description)/urdf/common.gazebo.xacro" />
-  <xacro:ur5_robot prefix="ur_arm_" joint_limited="true" kinematics_file="${load_yaml('$(arg kinematics_config)')}" />
+  <xacro:ur5_robot prefix="ur_arm_" />
 </robot>

File: ridgeback_ur_description/urdf/ridgeback_ur5_e_description.urdf.xacro (robot description, xacro)
@@ -1,13 +1,10 @@
 <?xml version="1.0"?>
 <robot xmlns:xacro="http://ros.org/wiki/xacro">
+  <xacro:include filename="$(find ur_description)/urdf/inc/ur5e_macro.xacro" />
   <joint name="arm_mount_joint" type="fixed">
-    <parent link="mid_mount" />
+    <parent link="top_plate_front_link" />
     <child link="ur_arm_base_link" />
-    <origin xyz="$(optenv RIDGEBACK_UR_XYZ 0.21 0.0 0.0)" rpy="$(optenv RIDGEBACK_UR_RPY 0 0 0)"/>
+    <origin xyz="$(optenv RIDGEBACK_UR_XYZ -0.105 0.0 0.0)" rpy="$(optenv RIDGEBACK_UR_RPY 0 0 3.1415927)"/>
   </joint>
-  <xacro:include filename="$(find ur_e_description)/urdf/ur5e.urdf.xacro" />
-  <xacro:arg name="kinematics_config" default="$(find ur_description)/config/ur5_e_default.yaml" />
-  <xacro:arg name="transmission_hw_interface" default="hardware_interface/PositionJointInterface"/>
-  <xacro:include filename="$(find ur_description)/urdf/common.gazebo.xacro" />
-  <xacro:ur5e_robot prefix="ur_arm_" joint_limited="true" kinematics_file="${load_yaml('$(arg kinematics_config)')}" />
+  <xacro:ur5e_robot prefix="ur_arm_" />
 </robot>

Commit message: Change default mount link of dual UR arms to tower_link

File: ridgeback_ur_description/urdf/ridgeback_dual_ur10_description.urdf.xacro (robot description, xacro)
@@ -3,12 +3,12 @@
   <xacro:include filename="$(find ur_description)/urdf/inc/ur10_macro.xacro" />
   <joint name="left_arm_mount_joint" type="fixed">
-    <parent link="left_arm_bulkhead_link" />
+    <parent link="tower_link" />
     <child link="left_ur_arm_base_link" />
-    <origin xyz="$(optenv RIDGEBACK_LEFT_UR_XYZ 0 0 0)" rpy="$(optenv RIDGEBACK_LEFT_UR_RPY 0 0 0)"/>
+    <origin xyz="$(optenv RIDGEBACK_LEFT_UR_XYZ 0 -0.3 0)" rpy="$(optenv RIDGEBACK_LEFT_UR_RPY 0 0 0)"/>
   </joint>
   <joint name="right_arm_mount_joint" type="fixed">
-    <parent link="right_arm_bulkhead_link" />
+    <parent link="tower_link" />
     <child link="right_ur_arm_base_link" />
-    <origin xyz="$(optenv RIDGEBACK_RIGHT_UR_XYZ 0 0 0)" rpy="$(optenv RIDGEBACK_RIGHT_UR_RPY 0 0 0)"/>
+    <origin xyz="$(optenv RIDGEBACK_RIGHT_UR_XYZ 0 0.1 0)" rpy="$(optenv RIDGEBACK_RIGHT_UR_RPY 0 0 0)"/>
   </joint>
   <xacro:ur10_robot prefix="right_ur_arm_" />

File: ridgeback_ur_description/urdf/ridgeback_dual_ur10_e_description.urdf.xacro (robot description, xacro)
@@ -3,12 +3,12 @@
   <xacro:include filename="$(find ur_description)/urdf/inc/ur10e_macro.xacro" />
   <joint name="left_arm_mount_joint" type="fixed">
-    <parent link="left_arm_bulkhead_link" />
+    <parent link="tower_link" />
     <child link="left_ur_arm_base_link" />
-    <origin xyz="$(optenv RIDGEBACK_LEFT_UR_XYZ 0 0 0)" rpy="$(optenv RIDGEBACK_LEFT_UR_RPY 0 0 0)"/>
+    <origin xyz="$(optenv RIDGEBACK_LEFT_UR_XYZ 0 -0.3 0)" rpy="$(optenv RIDGEBACK_LEFT_UR_RPY 0 0 0)"/>
   </joint>
   <joint name="right_arm_mount_joint" type="fixed">
-    <parent link="right_arm_bulkhead_link" />
+    <parent link="tower_link" />
     <child link="right_ur_arm_base_link" />
-    <origin xyz="$(optenv RIDGEBACK_RIGHT_UR_XYZ 0 0 0)" rpy="$(optenv RIDGEBACK_RIGHT_UR_RPY 0 0 0)"/>
+    <origin xyz="$(optenv RIDGEBACK_RIGHT_UR_XYZ 0 0.1 0)" rpy="$(optenv RIDGEBACK_RIGHT_UR_RPY 0 0 0)"/>
   </joint>
   <xacro:ur10e_robot prefix="right_ur_arm_" />

File: ridgeback_ur_description/urdf/ridgeback_dual_ur5_description.urdf.xacro (robot description, xacro)
@@ -3,12 +3,12 @@
   <xacro:include filename="$(find ur_description)/urdf/inc/ur5_macro.xacro" />
   <joint name="left_arm_mount_joint" type="fixed">
-    <parent link="left_arm_bulkhead_link" />
+    <parent link="tower_link" />
     <child link="left_ur_arm_base_link" />
-    <origin xyz="$(optenv RIDGEBACK_LEFT_UR_XYZ 0 0 0)" rpy="$(optenv RIDGEBACK_LEFT_UR_RPY 0 0 0)"/>
+    <origin xyz="$(optenv RIDGEBACK_LEFT_UR_XYZ 0 -0.3 0)" rpy="$(optenv RIDGEBACK_LEFT_UR_RPY 0 0 0)"/>
   </joint>
   <joint name="right_arm_mount_joint" type="fixed">
-    <parent link="right_arm_bulkhead_link" />
+    <parent link="tower_link" />
     <child link="right_ur_arm_base_link" />
-    <origin xyz="$(optenv RIDGEBACK_RIGHT_UR_XYZ 0 0 0)" rpy="$(optenv RIDGEBACK_RIGHT_UR_RPY 0 0 0)"/>
+    <origin xyz="$(optenv RIDGEBACK_RIGHT_UR_XYZ 0 0.1 0)" rpy="$(optenv RIDGEBACK_RIGHT_UR_RPY 0 0 0)"/>
   </joint>
   <xacro:ur5_robot prefix="right_ur_arm_" />

File: ridgeback_ur_description/urdf/ridgeback_dual_ur5_e_description.urdf.xacro (robot description, xacro)
@@ -3,12 +3,12 @@
   <xacro:include filename="$(find ur_description)/urdf/inc/ur5e_macro.xacro" />
   <joint name="left_arm_mount_joint" type="fixed">
-    <parent link="left_arm_bulkhead_link" />
+    <parent link="tower_link" />
     <child link="left_ur_arm_base_link" />
-    <origin xyz="$(optenv RIDGEBACK_LEFT_UR_XYZ 0 0 0)" rpy="$(optenv RIDGEBACK_LEFT_UR_RPY 0 0 0)"/>
+    <origin xyz="$(optenv RIDGEBACK_LEFT_UR_XYZ 0 -0.3 0)" rpy="$(optenv RIDGEBACK_LEFT_UR_RPY 0 0 0)"/>
   </joint>
   <joint name="right_arm_mount_joint" type="fixed">
-    <parent link="right_arm_bulkhead_link" />
+    <parent link="tower_link" />
     <child link="right_ur_arm_base_link" />
-    <origin xyz="$(optenv RIDGEBACK_RIGHT_UR_XYZ 0 0 0)" rpy="$(optenv RIDGEBACK_RIGHT_UR_RPY 0 0 0)"/>
+    <origin xyz="$(optenv RIDGEBACK_RIGHT_UR_XYZ 0 0.1 0)" rpy="$(optenv RIDGEBACK_RIGHT_UR_RPY 0 0 0)"/>
   </joint>
   <xacro:ur5e_robot prefix="right_ur_arm_" />

Commit message: Swap left and right arm positions; was incorrect previously

File: ridgeback_ur_description/urdf/ridgeback_dual_ur10_description.urdf.xacro (robot description, xacro)
@@ -5,10 +5,10 @@
     <parent link="tower_link" />
     <child link="left_ur_arm_base_link" />
-    <origin xyz="$(optenv RIDGEBACK_LEFT_UR_XYZ 0 -0.3 0)" rpy="$(optenv RIDGEBACK_LEFT_UR_RPY 0 0 0)"/>
+    <origin xyz="$(optenv RIDGEBACK_LEFT_UR_XYZ 0 0.1 0)" rpy="$(optenv RIDGEBACK_LEFT_UR_RPY 0 0 0)"/>
   </joint>
   <joint name="right_arm_mount_joint" type="fixed">
     <parent link="tower_link" />
     <child link="right_ur_arm_base_link" />
-    <origin xyz="$(optenv RIDGEBACK_RIGHT_UR_XYZ 0 0.1 0)" rpy="$(optenv RIDGEBACK_RIGHT_UR_RPY 0 0 0)"/>
+    <origin xyz="$(optenv RIDGEBACK_RIGHT_UR_XYZ 0 -0.3 0)" rpy="$(optenv RIDGEBACK_RIGHT_UR_RPY 0 0 0)"/>
   </joint>
   <xacro:ur10_robot prefix="right_ur_arm_" />

File: ridgeback_ur_description/urdf/ridgeback_dual_ur10_e_description.urdf.xacro (robot description, xacro)
@@ -5,10 +5,10 @@
     <parent link="tower_link" />
     <child link="left_ur_arm_base_link" />
-    <origin xyz="$(optenv RIDGEBACK_LEFT_UR_XYZ 0 -0.3 0)" rpy="$(optenv RIDGEBACK_LEFT_UR_RPY 0 0 0)"/>
+    <origin xyz="$(optenv RIDGEBACK_LEFT_UR_XYZ 0 0.1 0)" rpy="$(optenv RIDGEBACK_LEFT_UR_RPY 0 0 0)"/>
   </joint>
   <joint name="right_arm_mount_joint" type="fixed">
     <parent link="tower_link" />
     <child link="right_ur_arm_base_link" />
-    <origin xyz="$(optenv RIDGEBACK_RIGHT_UR_XYZ 0 0.1 0)" rpy="$(optenv RIDGEBACK_RIGHT_UR_RPY 0 0 0)"/>
+    <origin xyz="$(optenv RIDGEBACK_RIGHT_UR_XYZ 0 -0.3 0)" rpy="$(optenv RIDGEBACK_RIGHT_UR_RPY 0 0 0)"/>
   </joint>
   <xacro:ur10e_robot prefix="right_ur_arm_" />

File: ridgeback_ur_description/urdf/ridgeback_dual_ur5_description.urdf.xacro (robot description, xacro)
@@ -5,10 +5,10 @@
     <parent link="tower_link" />
     <child link="left_ur_arm_base_link" />
-    <origin xyz="$(optenv RIDGEBACK_LEFT_UR_XYZ 0 -0.3 0)" rpy="$(optenv RIDGEBACK_LEFT_UR_RPY 0 0 0)"/>
+    <origin xyz="$(optenv RIDGEBACK_LEFT_UR_XYZ 0 0.1 0)" rpy="$(optenv RIDGEBACK_LEFT_UR_RPY 0 0 0)"/>
   </joint>
   <joint name="right_arm_mount_joint" type="fixed">
     <parent link="tower_link" />
     <child link="right_ur_arm_base_link" />
-    <origin xyz="$(optenv RIDGEBACK_RIGHT_UR_XYZ 0 0.1 0)" rpy="$(optenv RIDGEBACK_RIGHT_UR_RPY 0 0 0)"/>
+    <origin xyz="$(optenv RIDGEBACK_RIGHT_UR_XYZ 0 -0.3 0)" rpy="$(optenv RIDGEBACK_RIGHT_UR_RPY 0 0 0)"/>
   </joint>
   <xacro:ur5_robot prefix="right_ur_arm_" />

File: ridgeback_ur_description/urdf/ridgeback_dual_ur5_e_description.urdf.xacro (robot description, xacro)
@@ -5,10 +5,10 @@
     <parent link="tower_link" />
     <child link="left_ur_arm_base_link" />
-    <origin xyz="$(optenv RIDGEBACK_LEFT_UR_XYZ 0 -0.3 0)" rpy="$(optenv RIDGEBACK_LEFT_UR_RPY 0 0 0)"/>
+    <origin xyz="$(optenv RIDGEBACK_LEFT_UR_XYZ 0 0.1 0)" rpy="$(optenv RIDGEBACK_LEFT_UR_RPY 0 0 0)"/>
   </joint>
   <joint name="right_arm_mount_joint" type="fixed">
     <parent link="tower_link" />
     <child link="right_ur_arm_base_link" />
-    <origin xyz="$(optenv RIDGEBACK_RIGHT_UR_XYZ 0 0.1 0)" rpy="$(optenv RIDGEBACK_RIGHT_UR_RPY 0 0 0)"/>
+    <origin xyz="$(optenv RIDGEBACK_RIGHT_UR_XYZ 0 -0.3 0)" rpy="$(optenv RIDGEBACK_RIGHT_UR_RPY 0 0 0)"/>
   </joint>
   <xacro:ur5e_robot prefix="right_ur_arm_" />
